Commit message: adjustment on wheel moment and mu

File: src/simulation/body_description/urdf/body.xacro (robot description, xacro)
@@ -8,5 +8,5 @@
   <xacro:property name="damping" value="0.7" />
   <xacro:property name="wheelmass" value="5" />
-  <xacro:property name="wheelmoment" value="0.006" />
+  <xacro:property name="wheelmoment" value="1" />
   <link name="base_link">
     <visual>
